Commit message: joint trajectory working

File: src/hitc_robot_description/urdf/hitc_robot_description.urdf (robot description, URDF)
Before this commit: robot hitc_robot_description, 3 links, 2 joints
Links:
- added link end_effector, mass 0.00358860280590412; collision mesh filename=package://hitc_robot_description/meshes/end_effector.STL; visual mesh filename=package://hitc_robot_description/meshes/end_effector.STL
- link link1: mass 1.72026759907067 -> 1.72026761826256
- link link2: mass 1.80507291432319 -> 1.8050728626833
Joints:
- added joint L2-EE: type continuous, parent link2, child end_effector, origin xyz=0.45 0 0 rpy=0 0 0, axis 0 0 -1
- joint L1-L2: axis 0 0 1 -> 0 0 -1; origin xyz=0.349999999999999 0 0 rpy=0 0 -1.5707963267949 -> xyz=0.35 0 0 rpy=0 0 1.5708
- joint base_L1: axis 0 0 1 -> 0 0 -1; origin xyz=0.12 0 0 rpy=0 0 1.02821445685467 -> xyz=0.12 0 0 rpy=0 0 -1.5708

Commit message: Float32MultiArray working on microRos

File: src/hitc_robot_description/urdf/hitc_robot_description.urdf (robot description, URDF)
Before this commit: robot hitc_robot_description, 4 links, 3 joints
Joints:
- joint L1-L2: axis 0 0 -1 -> 0 0 1
- joint L2-EE: axis 0 0 -1 -> 0 0 1
- joint base_L1: axis 0 0 -1 -> 0 0 1
